File: Projet_PAD_DDR/Projet_PAD_DDRV0.5.kicad_sch (KiCad schematic)
At the start: 54 parts, among them J1 USB_B_Micro, J2 Conn_02x07_Odd_Even, J3 Conn_01x02, J4 Conn_01x02, J5 Conn_01x02, J6 Conn_01x02, J7 Conn_01x08_Pin, J8 Conn_01x02_Pin, SW1 SW_MEC_5E, SW2 SW_MEC_5E, U1 STM32L476RGTx, U2 MCP1802x-xx02xOT, X1 MU00525-32.768K

Commit message: Version test première verification
Parts:
- removed C14: 1uF, Capacitor_SMD:C_0805_2012Metric_Pad1.18x1.45mm_HandSolder, symbol Device:C_Small
- removed D3: LED3, LED_SMD:LED_0805_2012Metric_Pad1.15x1.40mm_HandSolder, symbol Device:LED
- removed J7: Conn_01x08_Pin, Connector_PinHeader_2.54mm:PinHeader_1x08_P2.54mm_Vertical, symbol Connector:Conn_01x08_Pin
- removed J8: Conn_01x02_Pin, Connector_PinHeader_2.54mm:PinHeader_1x02_P2.54mm_Vertical, symbol Connector:Conn_01x02_Pin
- added C13: 100n, symbol Device:C_Small
- added C14, C19: C, symbol Device:C
- added C20, C21, C22, C23: C_Small, symbol Device:C_Small
- added R12, R13, R14, R18: R_Small, symbol Device:R_Small
- C1, C2: value 1uF -> C_Small; footprint Capacitor_SMD:C_0805_2012Metric_Pad1.18x1.45mm_HandSolder -> (none)
- C10, C11, C12, C15, C16, C17, C18, C24, C25, C3, C5, C6, C7, C8, C9: footprint Capacitor_SMD:C_0805_2012Metric_Pad1.18x1.45mm_HandSolder -> (none)
- C4: value 20pf -> 20p?; footprint Capacitor_SMD:C_0805_2012Metric_Pad1.18x1.45mm_HandSolder -> (none)
- D1: value LED1 -> LED; footprint LED_SMD:LED_0805_2012Metric_Pad1.15x1.40mm_HandSolder -> (none)
- D2: value LED2 -> LED; footprint LED_SMD:LED_0805_2012Metric_Pad1.15x1.40mm_HandSolder -> (none)
- H1, H2, H3, H4: footprint MountingHole:MountingHole_3.2mm_M3_DIN965_Pad -> (none)
- J1: footprint Connector_USB:USB_Micro-B_Wuerth_629105150521 -> (none)
- J2: footprint Connector_PinHeader_1.27mm:PinHeader_2x07_P1.27mm_Vertical_SMD -> (none)
- J3, J4, J5, J6: footprint Connector_JST:JST_XH_B2B-XH-A_1x02_P2.50mm_Vertical -> (none)
- R1: value 120 -> R_Small; footprint Resistor_SMD:R_0805_2012Metric_Pad1.20x1.40mm_HandSolder -> (none)
- R10, R5: value R_Cable_Right -> R_Small; footprint Resistor_SMD:R_0805_2012Metric_Pad1.20x1.40mm_HandSolder -> (none)
- R11: value 290 -> R_Small; footprint Resistor_SMD:R_0805_2012Metric_Pad1.20x1.40mm_HandSolder -> (none)
- R15, R2: footprint Resistor_SMD:R_0805_2012Metric_Pad1.20x1.40mm_HandSolder -> (none)
- R16: value 100 -> R_Small; footprint Resistor_SMD:R_0805_2012Metric_Pad1.20x1.40mm_HandSolder -> (none)
- R17: value 100k -> R_Small; footprint Resistor_SMD:R_0805_2012Metric_Pad1.20x1.40mm_HandSolder -> (none)
- R19: value 140 -> R_Small; footprint Resistor_SMD:R_0805_2012Metric_Pad1.20x1.40mm_HandSolder -> (none)
- R3, R7: value R_Cable_Up -> R_Small; footprint Resistor_SMD:R_0805_2012Metric_Pad1.20x1.40mm_HandSolder -> (none)
- R4, R8: value R_Cable_Down -> R_Small; footprint Resistor_SMD:R_0805_2012Metric_Pad1.20x1.40mm_HandSolder -> (none)
- R6, R9: value R_Cable_Left -> R_Small; footprint Resistor_SMD:R_0805_2012Metric_Pad1.20x1.40mm_HandSolder -> (none)
- SW1, SW2: footprint Button_Switch_SMD:SW_MEC_5GSH9 -> (none)
Connections:
- net +3.3V: now also C13.1
- net +5V: now also R18.2
- net GND: now also C13.2, C14.2, C19.2, C20.2, C21.2, C22.2, C23.2; no longer R11.1
- net PAD_ALIM: now also C14.1
- net LED_UP: now reaches U1.56 (PB4)
- net LED_DOWN: now reaches U1.57 (PB5)
- net LED_RIGHT: now reaches U1.58 (PB6)
- net LED_LEFT: now reaches U1.59 (PB7)
- net LED_ALIM: now reaches R11.2
- net LED_ALIM: now also C19.1, C20.1, C21.1, C22.1, C23.1, R12.2, R13.2, R14.2, R18.1
- new net LED_ALIM_DOWN: R12.1
- new net LED_ALIM_LEFT: R13.1
- new net LED_ALIM_RIGHT: R14.1
- new net LED_ALIM_UP: R11.1
- no-connect marks 44 -> 40
Other:
- note added: "Trou de Maintient"
- note removed: "Test pin"
- note removed: "Trou de montage"
- moved on the sheet: J3, J4, J5, J6, R17
