File: Projet_PAD_DDR/Projet_PAD_DDR.kicad_pcb (KiCad board)
At the start: 4 copper layers, 62 x 46 mm, 54 parts, among them J1 USB_B_Micro, J2 Conn_02x07_Odd_Even, J3 Conn_01x02, J4 Conn_01x02, J5 Conn_01x02, J6 Conn_01x02, J7 Conn_01x08_Pin, J8 Conn_01x02_Pin, SW1 SW_MEC_5E, SW2 SW_MEC_5E, U1 STM32L476RGTx, U2 MCP1802x-xx02xOT, X1 MU00525-32.768K

Commit message: Version a verifier
Parts:
- added J9: Conn_01x02_Pin, Connector_PinHeader_2.54mm:PinHeader_1x02_P2.54mm_Vertical, F.Cu at (234.1, 115.4)
- added Q1: BCX56, Package_TO_SOT_SMD:SOT-223, F.Cu at (196.6, 143.6)
- added R12: 100k, Resistor_SMD:R_0805_2012Metric_Pad1.20x1.40mm_HandSolder, F.Cu at (197.8, 135.9)
- moved R1 21.2 mm to (200.5, 117.4), turned to -90 degrees
- moved D1 17.4 mm to (200.5, 121.2), turned to 90 degrees
- moved R17 8.53 mm to (194.9, 137.7), turned to 180 degrees
- moved C10 4.08 mm to (207.3, 140.9), turned to 0 degrees
- moved C2 1.76 mm to (201.6, 142.4), turned to -90 degrees
- moved C1 1.02 mm to (201.4, 146.5), turned to 90 degrees
- moved J1 0.40 mm to (207.9, 153.6)
- moved C14 0.38 mm to (201.5, 150.6)
Connections:
- C15 pad 1: PAD_ALIM -> Net-(C15-Pad1)
- C16 pad 1: PAD_ALIM -> Net-(C15-Pad1)
- C17 pad 1: PAD_ALIM -> Net-(C15-Pad1)
- C18 pad 1: PAD_ALIM -> Net-(C15-Pad1)
- R10 pad 2: PAD_ALIM -> Net-(C15-Pad1)
- R17 pad 1: +3.3V -> PAD_ALIM
- R17 pad 2: PAD_ALIM -> GND
- R7 pad 2: PAD_ALIM -> Net-(C15-Pad1)
- R8 pad 2: PAD_ALIM -> Net-(C15-Pad1)
- R9 pad 2: PAD_ALIM -> Net-(C15-Pad1)
- U1 pad 40: unconnected-(U1-PC9-Pad40) -> Commande transistor
Routing:
- net Net-(C15-Pad1): track 0.00 -> 108.2 mm, vias 0 -> 4
- net PAD_ALIM: track 107.2 -> 6.06 mm, vias 4 -> 0
- net USART2_RX: track 17.4 -> 45.2 mm, vias 2 -> 4
- net USART2_TX: track 15.2 -> 39.3 mm, vias 2 -> 4
- net Commande transistor: track 0.00 -> 17.2 mm
- net +5V: track 18.9 -> 30.2 mm
- net GND: track 30.8 -> 27.6 mm, vias 23 -> 24
- net +3.3V: track 39.1 -> 36.5 mm, vias 8 -> 9
- net BUTTON: track 35.7 -> 36.5 mm
- net PAD_ALIM_UP: track 48.4 -> 47.7 mm
