File: Projet_PAD_DDR/Projet_PAD_DDR.kicad_sch (KiCad schematic)
At the start: 54 parts, among them J1 USB_B_Micro, J2 Conn_02x07_Odd_Even, J3 Conn_01x02, J4 Conn_01x02, J5 Conn_01x02, J6 Conn_01x02, J7 Conn_01x08_Pin, J8 Conn_01x02_Pin, SW1 SW_MEC_5E, SW2 SW_MEC_5E, U1 STM32L476RGTx, U2 MCP1802x-xx02xOT, X1 MU00525-32.768K

Commit message: Version a verifier
Parts:
- added J9: Conn_01x02_Pin, Connector_PinHeader_2.54mm:PinHeader_1x02_P2.54mm_Vertical, symbol Connector:Conn_01x02_Pin
- added Q1: BCX56, Package_TO_SOT_SMD:SOT-223, symbol Transistor_BJT:BCX56
- added R12: 100k, Resistor_SMD:R_0805_2012Metric_Pad1.20x1.40mm_HandSolder, symbol Device:R_Small
Connections:
- net +3.3V: no longer R17.1
- net +5V: now also Q1.2 (C)
- net GND: now also R17.2
- net PAD_ALIM: now also R17.1, Q1.3 (E), R12.1; no longer C15.1, C16.1, C17.1, C18.1, R10.2, R17.2, R7.2, R8.2, R9.2
- net USART2_RX: now also J9.2 (Pin_2)
- net USART2_TX: now also J9.1 (Pin_1)
- net Commande transistor: now reaches U1.40 (PC9)
- net Commande transistor: now also Q1.1 (B)
- new net: C15.1, C16.1, C17.1, C18.1, R10.2, R12.2, R7.2, R8.2, R9.2
- no-connect marks 44 -> 43
Other:
- note added: "Securite alim"
- moved on the sheet: R17
