File: v3/V3.kicad_pcb (KiCad board)
At the start: 4 copper layers, 42 x 42.5 mm, 64 parts, among them J1 Conn_01x02_Pin, J10 USB_C_Receptacle_USB2.0_16P, J11 Conn_01x02_Pin, J12 Conn_01x02_Pin, J13 Conn_01x02_Pin, J14 Conn_01x02_Pin, J2 Conn_02x07_Odd_Even, J3 Conn_01x02, J4 Conn_01x02, J5 Conn_01x02, J6 Conn_01x02, J7 Conn_01x02_Pin, J8 Conn_01x02_Pin, J9 Conn_01x02_Pin, Q1 BCX56, U1 STM32G431K6Tx, U2 MCP1802x-xx02xOT, X1 MU00525-32.768K

Commit message: Version final
Parts:
- R12: value 100k -> 4k7
- R13, R14, R18, R20: value 4k7 -> 100K
Other:
- board text added: "Down"
- board text added: "Left"
- board text added: "Right"
- board text added: "UP"
Changed lines of the file:
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@@
 			)
 		)
-		(property "Value" "4k7"
+		(property "Value" "100K"
 			(at 0 -1.65 90)
 			(layer "B.Fab")
@@
 			)
 		)
-		(property "Value" "100k"
+		(property "Value" "4k7"
 			(at 0 -1.65 0)
 			(layer "B.Fab")
@@
 			)
 		)
-		(property "Value" "4k7"
+		(property "Value" "100K"
 			(at 0 -1.65 90)
 			(layer "B.Fab")
@@
 			)
 		)
-		(property "Value" "4k7"
+		(property "Value" "100K"
 			(at 0 -1.65 90)
 			(layer "B.Fab")
@@
 			)
 		)
-		(property "Value" "4k7"
+		(property "Value" "100K"
 			(at 0 -1.65 90)
 			(layer "B.Fab")
@@
 		)
 	)
+	(gr_text "Down"
+		(at 225.6 150.6 0)
+		(layer "F.SilkS")
+		(effects
+			(font
+				(size 0.8 0.8)
+				(thickness 0.16)
+				(bold yes)
+			)
+			(justify left bottom)
+		)
+	)
+	(gr_text "Right"
+		(at 219.8 134.2 0)
+		(layer "F.SilkS")
+		(effects
+			(font
+				(size 0.8 0.8)
+				(thickness 0.16)
+				(bold yes)
+			)
+			(justify left bottom)
+		)
+	)
+	(gr_text "UP"
+		(at 213.2 126.2 0)
+		(layer "F.SilkS")
+		(effects
+			(font
+				(size 0.8 0.8)
+				(thickness 0.16)
+				(bold yes)
+			)
+			(justify left bottom)
+		)
+	)
+	(gr_text "Left"
+		(at 194.4 143.2 0)
+		(layer "F.SilkS")
+		(effects
+			(font
+				(size 0.8 0.8)
+				(thickness 0.16)
+				(bold yes)
+			)
+			(justify left bottom)
+		)
+	)
 	(gr_text "G/A"
 		(at 227 135.62 90)
@@
 	)
 	(gr_text "G/A"
-		(at 224.3 144.56 0)
+		(at 224.3 144.8 0)
 		(layer "F.SilkS")
 		(effects

Commit message: Version final + seri
Parts:
- J10: footprint Connector_USB:USB_C_Receptacle_GCT_USB4105-xx-A_16P_TopMnt_Horizontal -> Connector_USB:USB_C_Receptacle_HRO_TYPE-C-31-M-12
- moved J1 0.44 mm to (196.4, 148.9)
Routing:
- net PAD_ALIM_UP: track 16.6 -> 17.3 mm
- net GND: vias 6 -> 12
Other:
- board text added: "FG.Sourbé M.Sayavong M.Dalmon S.Drault"
